File: Revision History.kicad_sch (KiCad schematic)
At the start: 0 parts

Commit message: Outputs generated, ready for prototyping
Changed lines of the file:
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@@
 		)
 	)
-	(text_box "- _________________________________\n\n- _________________________________\n\n- _________________________________\n\n- _________________________________\n\n- _________________________________\n\n- _________________________________\n\n- _________________________________\n\n- _________________________________\n\n- _________________________________\n\n- _________________________________\n\n- _________________________________\n\n- _________________________________\n\n- _________________________________\n\n- _________________________________\n\n- _________________________________\n\n- _________________________________\n\n- _________________________________"
+	(text_box "- Board Creation on Kicad\n\n- _________________________________\n\n- _________________________________\n\n- _________________________________\n\n- _________________________________\n\n- _________________________________\n\n- _________________________________\n\n- _________________________________\n\n- _________________________________\n\n- _________________________________\n\n- _________________________________\n\n- _________________________________\n\n- _________________________________\n\n- _________________________________\n\n- _________________________________\n\n- _________________________________\n\n- _________________________________"
 		(exclude_from_sim no)
 		(at 22.86 40.64 0)
@@
 		(stroke
 			(width -0.0001)
-			(type default)
+			(type solid)
 		)
 		(fill
@@
 		)
 	)
-	(text_box "DD.MM.YYYY - xxx Revision\nVariant: xxx"
+	(text_box "01.04.2025 - V1 Revision\nVariant: No Variant"
 		(exclude_from_sim no)
 		(at 20.32 31.75 0)
@@
 		(stroke
 			(width -0.0001)
-			(type default)
+			(type solid)
 		)
 		(fill
