File: PowMon.kicad_pcb (KiCad board)
At the start: 2 copper layers, 34 x 40 mm, 37 parts, among them J2 1x3 pin vertical, J3 1x3 pin vertical, J4 1x3 pin vertical, J5 1x3 pin vertical, J6 22-28-6040, J7 22-28-6040, P1 5KEV-0, P2 5KEV-0, T1 NSI50010YT1G, U1 INA226

Commit message: Intermediary save
Parts:
- added kibuzzard-67FD6413: G***, kibuzzard-67FD6413, F.Cu at (120.0, 106.5)
- added kibuzzard-67FD642C: G***, kibuzzard-67FD642C, F.Cu at (120.0, 114.0)
- added kibuzzard-67FD645D: G***, kibuzzard-67FD645D, F.Cu at (141.0, 106.5)
- added kibuzzard-67FD646E: G***, kibuzzard-67FD646E, F.Cu at (141.0, 114.0)
Other:
- board text removed: "G"
- board text removed: "V"
